File: hardware/r2_pico_carrier/r2_pico_carrier.kicad_sch (KiCad schematic)
At the start: 63 parts, among them J1 5V in, J2 OLED SSD1306, SW1 display, U1 PCA9517A

Commit message: Carrier board: PCA9517A port A (no offset) on the long cables; README warns about Pico orientation, terminal wiring with USB in, SW1 rotation
Parts:
- JP1, JP2: LCSC C49661 -> C50984
Connections:
- net SCL: now also U1.7 (SCLB); no longer U1.2 (SCLA)
- net SCL_L: now also U1.2 (SCLA); no longer U1.7 (SCLB)
- net SDA: now also U1.6 (SDAB); no longer U1.3 (SDAA)
- net SDA_L: now also U1.3 (SDAA); no longer U1.6 (SDAB)
Changed lines of the file:
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@@
 (kicad_sch (version 20250114) (generator "r2_pico_carrier_gen") (generator_version "10.0") (paper "A3") (title_block (title "R2 Pico carrier") (date "2026-10-27") (rev "A") (company "ROS2D2 · Astromech Spain") (comment 1 "Generated by gen/make_sch.py from gen/parts.py"))
-(symbol (lib_id "Connector_Generic:Conn_01x20") (at 39.37 124.46 0) (unit 1) (exclude_from_sim no) (in_bom yes) (on_board yes) (dnp no) (property "Reference" "JP1" (at 42.37 120.46000000000001 0) (effects (font (size 1.27 1.27)))) (property "Value" "Pico 2 pins 1-20" (at 42.37 122.96000000000001 0) (effects (font (size 1.27 1.27)))) (property "Footprint" "Connector_PinSocket_2.54mm:PinSocket_1x20_P2.54mm_Vertical" (at 42.37 125.46000000000001 0) (effects (font (size 1.27 1.27)) (hide yes))) (property "Datasheet" "" (at 42.37 127.96000000000001 0) (effects (font (size 1.27 1.27)) (hide yes))) (property "LCSC" "C49661" (at 42.37 130.46 0) (effects (font (size 1.27 1.27)) (hide yes))) (pin "1") (pin "2") (pin "3") (pin "4") (pin "5") (pin "6") (pin "7") (pin "8") (pin "9") (pin "10") (pin "11") (pin "12") (pin "13") (pin "14") (pin "15") (pin "16") (pin "17") (pin "18") (pin "19") (pin "20") (instances (project "r2_pico_carrier" (path "/1e5ddbbd-1ed4-52be-93d8-b73224ab9bea" (reference "JP1") (unit 1)))))
+(symbol (lib_id "Connector_Generic:Conn_01x20") (at 39.37 124.46 0) (unit 1) (exclude_from_sim no) (in_bom yes) (on_board yes) (dnp no) (property "Reference" "JP1" (at 42.37 120.46000000000001 0) (effects (font (size 1.27 1.27)))) (property "Value" "Pico 2 pins 1-20" (at 42.37 122.96000000000001 0) (effects (font (size 1.27 1.27)))) (property "Footprint" "Connector_PinSocket_2.54mm:PinSocket_1x20_P2.54mm_Vertical" (at 42.37 125.46000000000001 0) (effects (font (size 1.27 1.27)) (hide yes))) (property "Datasheet" "" (at 42.37 127.96000000000001 0) (effects (font (size 1.27 1.27)) (hide yes))) (property "LCSC" "C50984" (at 42.37 130.46 0) (effects (font (size 1.27 1.27)) (hide yes))) (pin "1") (pin "2") (pin "3") (pin "4") (pin "5") (pin "6") (pin "7") (pin "8") (pin "9") (pin "10") (pin "11") (pin "12") (pin "13") (pin "14") (pin "15") (pin "16") (pin "17") (pin "18") (pin "19") (pin "20") (instances (project "r2_pico_carrier" (path "/1e5ddbbd-1ed4-52be-93d8-b73224ab9bea" (reference "JP1") (unit 1)))))
 (no_connect (at 34.29 101.60))
 (no_connect (at 34.29 104.14))
@@
 (global_label "TRIG3" (shape passive) (at 34.29 147.32 180) (fields_autoplaced yes) (effects (font (size 1.27 1.27)) (justify right)))
 (global_label "ECHO3_P" (shape passive) (at 34.29 149.86 180) (fields_autoplaced yes) (effects (font (size 1.27 1.27)) (justify right)))
-(symbol (lib_id "Connector_Generic:Conn_01x20") (at 95.25 124.46 0) (unit 1) (exclude_from_sim no) (in_bom yes) (on_board yes) (dnp no) (property "Reference" "JP2" (at 98.25 120.46000000000001 0) (effects (font (size 1.27 1.27)))) (property "Value" "Pico 2 pins 40-21" (at 98.25 122.96000000000001 0) (effects (font (size 1.27 1.27)))) (property "Footprint" "Connector_PinSocket_2.54mm:PinSocket_1x20_P2.54mm_Vertical" (at 98.25 125.46000000000001 0) (effects (font (size 1.27 1.27)) (hide yes))) (property "Datasheet" "" (at 98.25 127.96000000000001 0) (effects (font (size 1.27 1.27)) (hide yes))) (property "LCSC" "C49661" (at 98.25 130.46 0) (effects (font (size 1.27 1.27)) (hide yes))) (pin "1") (pin "2") (pin "3") (pin "4") (pin "5") (pin "6") (pin "7") (pin "8") (pin "9") (pin "10") (pin "11") (pin "12") (pin "13") (pin "14") (pin "15") (pin "16") (pin "17") (pin "18") (pin "19") (pin "20") (instances (project "r2_pico_carrier" (path "/1e5ddbbd-1ed4-52be-93d8-b73224ab9bea" (reference "JP2") (unit 1)))))
+(symbol (lib_id "Connector_Generic:Conn_01x20") (at 95.25 124.46 0) (unit 1) (exclude_from_sim no) (in_bom yes) (on_board yes) (dnp no) (property "Reference" "JP2" (at 98.25 120.46000000000001 0) (effects (font (size 1.27 1.27)))) (property "Value" "Pico 2 pins 40-21" (at 98.25 122.96000000000001 0) (effects (font (size 1.27 1.27)))) (property "Footprint" "Connector_PinSocket_2.54mm:PinSocket_1x20_P2.54mm_Vertical" (at 98.25 125.46000000000001 0) (effects (font (size 1.27 1.27)) (hide yes))) (property "Datasheet" "" (at 98.25 127.96000000000001 0) (effects (font (size 1.27 1.27)) (hide yes))) (property "LCSC" "C50984" (at 98.25 130.46 0) (effects (font (size 1.27 1.27)) (hide yes))) (pin "1") (pin "2") (pin "3") (pin "4") (pin "5") (pin "6") (pin "7") (pin "8") (pin "9") (pin "10") (pin "11") (pin "12") (pin "13") (pin "14") (pin "15") (pin "16") (pin "17") (pin "18") (pin "19") (pin "20") (instances (project "r2_pico_carrier" (path "/1e5ddbbd-1ed4-52be-93d8-b73224ab9bea" (reference "JP2") (unit 1)))))
 (no_connect (at 90.17 101.60))
 (global_label "VSYS" (shape passive) (at 90.17 104.14 180) (fields_autoplaced yes) (effects (font (size 1.27 1.27)) (justify right)))
@@
 (symbol (lib_id "Logic_LevelTranslator:TCA9517ADGK") (at 280.67 44.45 0) (unit 1) (exclude_from_sim no) (in_bom yes) (on_board yes) (dnp no) (property "Reference" "U1" (at 283.67 40.45 0) (effects (font (size 1.27 1.27)))) (property "Value" "PCA9517A" (at 283.67 42.95 0) (effects (font (size 1.27 1.27)))) (property "Footprint" "Package_SO:VSSOP-8_3x3mm_P0.65mm" (at 283.67 45.45 0) (effects (font (size 1.27 1.27)) (hide yes))) (property "Datasheet" "" (at 283.67 47.95 0) (effects (font (size 1.27 1.27)) (hide yes))) (property "LCSC" "C80799" (at 283.67 50.45 0) (effects (font (size 1.27 1.27)) (hide yes))) (pin "1") (pin "2") (pin "3") (pin "4") (pin "5") (pin "6") (pin "7") (pin "8") (instances (project "r2_pico_carrier" (path "/1e5ddbbd-1ed4-52be-93d8-b73224ab9bea" (reference "U1") (unit 1)))))
 (global_label "+3V3" (shape passive) (at 278.13 31.75 90) (fields_autoplaced yes) (effects (font (size 1.27 1.27)) (justify left)))
-(global_label "SCL" (shape passive) (at 267.97 41.91 180) (fields_autoplaced yes) (effects (font (size 1.27 1.27)) (justify right)))
-(global_label "SDA" (shape passive) (at 267.97 46.99 180) (fields_autoplaced yes) (effects (font (size 1.27 1.27)) (justify right)))
+(global_label "SCL_L" (shape passive) (at 267.97 41.91 180) (fields_autoplaced yes) (effects (font (size 1.27 1.27)) (justify right)))
+(global_label "SDA_L" (shape passive) (at 267.97 46.99 180) (fields_autoplaced yes) (effects (font (size 1.27 1.27)) (justify right)))
 (global_label "GND" (shape passive) (at 280.67 57.15 270) (fields_autoplaced yes) (effects (font (size 1.27 1.27)) (justify right)))
 (global_label "+3V3" (shape passive) (at 293.37 52.07 0) (fields_autoplaced yes) (effects (font (size 1.27 1.27)) (justify left)))
-(global_label "SDA_L" (shape passive) (at 293.37 46.99 0) (fields_autoplaced yes) (effects (font (size 1.27 1.27)) (justify left)))
-(global_label "SCL_L" (shape passive) (at 293.37 41.91 0) (fields_autoplaced yes) (effects (font (size 1.27 1.27)) (justify left)))
+(global_label "SDA" (shape passive) (at 293.37 46.99 0) (fields_autoplaced yes) (effects (font (size 1.27 1.27)) (justify left)))
+(global_label "SCL" (shape passive) (at 293.37 41.91 0) (fields_autoplaced yes) (effects (font (size 1.27 1.27)) (justify left)))
 (global_label "+3V3" (shape passive) (at 283.21 31.75 90) (fields_autoplaced yes) (effects (font (size 1.27 1.27)) (justify left)))
 (symbol (lib_id "Device:C") (at 308.61 44.45 0) (unit 1) (exclude_from_sim no) (in_bom yes) (on_board yes) (dnp no) (property "Reference" "C5" (at 311.61 40.45 0) (effects (font (size 1.27 1.27)))) (property "Value" "100n" (at 311.61 42.95 0) (effects (font (size 1.27 1.27)))) (property "Footprint" "Capacitor_SMD:C_0603_1608Metric" (at 311.61 45.45 0) (effects (font (size 1.27 1.27)) (hide yes))) (property "Datasheet" "" (at 311.61 47.95 0) (effects (font (size 1.27 1.27)) (hide yes))) (property "LCSC" "C14663" (at 311.61 50.45 0) (effects (font (size 1.27 1.27)) (hide yes))) (pin "1") (pin "2") (instances (project "r2_pico_carrier" (path "/1e5ddbbd-1ed4-52be-93d8-b73224ab9bea" (reference "C5") (unit 1)))))

Commit message: Carrier board: OLED (HS96L03W2C03) fitted at the factory, lying flat; round Astromech Spain logo; 80 x 90 mm
Parts:
- added H5, H6, H7, H8: M2 OLED, MountingHole:MountingHole_2.2mm_M2, symbol Mechanical:MountingHole
- J2: value OLED SSD1306 -> OLED HS96L03W2C03; footprint Connector_PinSocket_2.54mm:PinSocket_1x04_P2.54mm_Vertical -> Connector_PinHeader_2.54mm:PinHeader_1x04_P2.54mm_Vertical; LCSC C2718488 -> C5248080
Other:
- moved on the sheet: H1, H2, H3, H4
