File: hardware/r2_pico_carrier/r2_pico_carrier.kicad_pcb (KiCad board)
At the start: 2 copper layers, 80 x 90 mm, 70 parts, among them J1 5V in, J2 OLED header, J3 Qwiic, J4 expansion, J5 USB-C 5V in, SW1 display, U1 PCA9517A

Commit message: Carrier board, pre-order review: U1 (PCA9517A) +270 in the JLC CPL; J1 turned so its wires enter from the left edge; USB-C J5 flush with the edge; PCBWay maker for C14663; README viewer checks
Parts:
- moved J1 6.33 mm to (5.60, 59.0), turned to -90 degrees
- moved J5 0.40 mm to (3.60, 75.0)
Routing:
- net XSHUT4: track 69.0 -> 51.1 mm, vias 2 -> 0
- net ECHO2_P: track 43.7 -> 30.9 mm
- net SDA: track 117.3 -> 106.8 mm, vias 1 -> 3
- net STAT3: track 30.1 -> 38.4 mm
- net SDA_L: track 27.0 -> 34.4 mm, vias 0 -> 1
- net GND: track 483.0 -> 490.1 mm, vias 3 -> 5
- net ECHO4_P: track 37.9 -> 44.1 mm, vias 1 -> 2
- net XSHUT3: track 52.7 -> 47.1 mm
- net CC1: track 2.44 -> 6.55 mm, vias 0 -> 2
- net STAT7: track 14.6 -> 10.9 mm, vias 1 -> 0
- net STAT2: track 29.1 -> 31.9 mm
- net STAT4: track 52.9 -> 55.7 mm
- net SCL: track 103.7 -> 106.3 mm, vias 3 -> 2
- net 5V_IN: track 18.9 -> 21.4 mm
- net ECHO3_P: track 38.1 -> 40.4 mm
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Other:
- board text added: "+5V"
- board text added: "GND"
- board text removed: "+5V GND"

Commit message: Carrier board: all four VL53L0X behind the U1 repeater (any VL connector, cables up to 1 m; Pico bus keeps display, Qwiic, EXP); EXP header moved left, 3.4 mm clear of the OLED
Parts:
- moved J4 3.00 mm to (27.5, 69.0)
Connections:
- VL1 pad 3: SCL -> SCL_L
- VL1 pad 4: SDA -> SDA_L
- VL2 pad 3: SCL -> SCL_L
- VL2 pad 4: SDA -> SDA_L
Routing:
- net SDA: track 106.8 -> 160.4 mm, vias 3 -> 0
- net SCL: track 106.3 -> 156.5 mm, vias 2 -> 0
- net +3V3: track 123.9 -> 149.6 mm
- net SDA_L: track 34.4 -> 57.0 mm
- net XSHUT3: track 47.1 -> 67.2 mm
- net SCL_L: track 28.2 -> 47.5 mm
- net XSHUT4: track 51.1 -> 70.1 mm, vias 0 -> 1
- net GND: track 490.1 -> 499.4 mm
- net +5V: track 101.6 -> 110.5 mm, vias 0 -> 2
- net STAT3: track 38.4 -> 30.2 mm
- net ECHO2_P: track 30.9 -> 38.6 mm
- net ECHO3_P: track 40.4 -> 33.1 mm, vias 1 -> 2
- net CC2: track 2.91 -> 10.1 mm, vias 0 -> 2
- net TRIG3: track 40.5 -> 33.8 mm, vias 0 -> 1
- net ECHO1_P: track 41.7 -> 35.8 mm
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Other:
- board text added: "cable <= 1 m"
- board text removed: "< 50 cm"
- board text removed: "> 50 cm"
